File: cubesatsim/cubesatsim-hat/cubesatsim-hat.kicad_sch (KiCad schematic)
At the start: 15 parts, among them J1 GPIO, J8 Conn_01x17_Pin, SW1 SW_SPST

Commit message: stuff
Parts:
- removed J8: Conn_01x17_Pin, Connector_PinHeader_1.27mm:PinHeader_1x17_P1.27mm_Horizontal, symbol Connector:Conn_01x17_Pin
- removed SW1: SW_SPST, Button_Switch_SMD:SW_Push_1P1T_NO_6x6mm_H9.5mm, symbol Switch:SW_Push
- added D1: D, Diode_SMD:D_0201_0603Metric, symbol Device:D
- added J2: 3 pin conn, Connector_PinHeader_1.27mm:PinHeader_1x03_P1.27mm_Vertical, symbol Connector:Conn_01x03_Pin
- added J3: Fan 2, Connector_PinHeader_1.27mm:PinHeader_1x02_P1.27mm_Vertical, symbol Connector:Conn_01x02_Pin
- added J4: Sensor ADC Connection, Connector_PinHeader_1.27mm:PinHeader_1x02_P1.27mm_Vertical, symbol Connector:Conn_01x02_Pin
- added J5: SPST External, Connector_PinHeader_1.27mm:PinHeader_1x02_P1.27mm_Vertical, symbol Connector:Conn_01x02_Pin
- added J6: LED Connections, Connector_PinHeader_1.27mm:PinHeader_1x06_P1.27mm_Vertical, symbol Connector:Conn_01x06_Pin
- added J7: Fan 1, Connector_PinHeader_1.27mm:PinHeader_1x02_P1.27mm_Vertical, symbol Connector:Conn_01x02_Pin
- added SW1: SW_SPST, Button_Switch_SMD:SW_DIP_SPSTx01_Slide_6.7x4.1mm_W8.61mm_P2.54mm_LowProfile, symbol Switch:SW_SPST
- renumbered R5 to R3, R9 to R4, R3 to R5, R7 to R6, R4 to R7, R6 to R9
Connections:
- net at J1.10 (Pin_10): now also J2.1 (Pin_1)
- net at J1.14 (Pin_14): now also J5.2 (Pin_2), SW1.1 (A)
- net at R4.1, R5.1: now also J1.22 (Pin_22); no longer J1.15 (Pin_15)
- net at J1.18 (Pin_18): now also J5.1 (Pin_1), SW1.2 (B)
- net at D2.1 (K), D3.1 (K), D4.1 (K)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: now also J4.1 (Pin_1), J6.1 (Pin_1), J6.3 (Pin_3), J6.5 (Pin_5)
- net at J1.6 (Pin_6): now also J2.3 (Pin_3), J3.1 (Pin_1), J7.1 (Pin_1)
- net at J1.8 (Pin_8): now also J2.2 (Pin_2)
- net at R2.2, R3.1: now also D1.2 (A)
- net at R9.2: now also J6.2 (Pin_2)
- net at R7.2: now also J6.4 (Pin_4)
- net at R1.2: now also J3.2 (Pin_2), J7.2 (Pin_2)
- net at R5.2: now also J6.6 (Pin_6)
- new net: D1.1 (K), J4.2 (Pin_2)
Other:
- note added: "LED1"
- note added: "LED2"
- note added: "LED3"
- note added: "gnd"
