File: sensor-hat/cubesatsim-hat.kicad_pcb (KiCad board)
At the start: 2 copper layers, 65 x 56 mm, 25 parts, among them J1 GPIO, J2 3 pin conn, J3 Fan 2, J4 Sensor ADC Connection, J5 SPST External, J6 LED Connections, J7 Fan 1, SW1 SW_SPST

Commit message: stuff
Parts:
- removed D1: D, Diode_SMD:D_0201_0603Metric
- removed J2: 3 pin conn, Connector_PinHeader_1.27mm:PinHeader_1x03_P1.27mm_Vertical
- removed J3: Fan 2, Connector_PinHeader_1.27mm:PinHeader_1x02_P1.27mm_Vertical
- removed J4: Sensor ADC Connection, Connector_PinHeader_1.27mm:PinHeader_1x02_P1.27mm_Vertical
- removed J5: SPST External, Connector_PinHeader_1.27mm:PinHeader_1x02_P1.27mm_Vertical
- removed J6: LED Connections, Connector_PinHeader_1.27mm:PinHeader_1x06_P1.27mm_Vertical
- removed J7: Fan 1, Connector_PinHeader_1.27mm:PinHeader_1x02_P1.27mm_Vertical
- removed MH3, MH4: MountingHole_2.7mm_M2.5, MountingHole:MountingHole_2.7mm_M2.5
- added J8: Conn_01x17_Pin, Connector_PinHeader_1.27mm:PinHeader_1x17_P1.27mm_Horizontal, F.Cu at (133.8, 66.0)
- R3: value 10000 -> 1000
- R5: value 1000 -> 10000
- SW1: footprint Button_Switch_SMD:SW_DIP_SPSTx01_Slide_6.7x4.1mm_W8.61mm_P2.54mm_LowProfile -> Button_Switch_SMD:SW_Push_1P1T_NO_6x6mm_H9.5mm
- moved D2 45.4 mm to (153.0, 64.5), turned to 0 degrees
- moved D3 38.8 mm to (148.0, 64.5), turned to 0 degrees
- moved R9 38.5 mm to (155.5, 58.5), turned to -90 degrees
- moved SW1 37.9 mm to (110.2, 57.5), turned to -90 degrees
- moved R8 34.1 mm to (150.5, 58.5), turned to 90 degrees
- moved D4 33.9 mm to (143.0, 64.5), turned to 0 degrees
- moved R7 30.2 mm to (145.5, 58.5), turned to -90 degrees
- moved R4 24.2 mm to (130.0, 59.0), turned to -90 degrees
- moved R5 22.9 mm to (132.5, 59.0), turned to -90 degrees
- moved R6 22.4 mm to (135.0, 59.0), turned to -90 degrees
- moved R1 16.0 mm to (122.5, 59.0), turned to -90 degrees
- moved R2 5.03 mm to (125.0, 59.0)
- moved R3 0.76 mm to (127.5, 59.0)
Connections:
- J1 pad 15: unconnected-(J1-Pin_15-Pad15) -> Net-(J1-Pin_15)
- J1 pad 22: Net-(J1-Pin_22) -> unconnected-(J1-Pin_22-Pad22)
- R2 pad 2: Net-(D1-A) -> Net-(J8-Pin_8)
- R3 pad 1: Net-(D1-A) -> Net-(J1-Pin_15)
- R3 pad 2: Net-(D2-K) -> Net-(J8-Pin_6)
- R4 pad 1: Net-(J1-Pin_22) -> Net-(J1-Pin_28)
- R4 pad 2: Net-(D2-A) -> Net-(J8-Pin_4)
- R5 pad 1: Net-(J1-Pin_22) -> Net-(J8-Pin_8)
- R5 pad 2: Net-(J6-Pin_6) -> Net-(D2-K)
- R6 pad 1: Net-(J1-Pin_28) -> Net-(J1-Pin_36)
- R6 pad 2: Net-(D4-A) -> Net-(J8-Pin_2)
- R7 pad 2: Net-(J6-Pin_4) -> Net-(D4-A)
- R9 pad 1: Net-(J1-Pin_36) -> Net-(J1-Pin_15)
- R9 pad 2: Net-(J6-Pin_2) -> Net-(D2-A)
- SW1 pad 1: Net-(J1-Pin_14) -> Net-(J1-Pin_18)
- SW1 pad 2: Net-(J1-Pin_18) -> Net-(J1-Pin_14)
Routing:
- net Net-(D2-K): track 0.00 -> 55.7 mm
- net Net-(J1-Pin_18): track 0.00 -> 50.5 mm
- net Net-(J1-Pin_14): track 0.00 -> 45.3 mm
- net Net-(J1-Pin_15): track 0.00 -> 41.1 mm
- net Net-(J1-Pin_6): track 0.00 -> 35.1 mm
- net Net-(J1-Pin_36): track 0.00 -> 27.3 mm
- net Net-(J1-Pin_28): track 0.00 -> 26.6 mm
- net Net-(J1-Pin_10): track 0.00 -> 21.8 mm
- net Net-(J1-Pin_8): track 0.00 -> 21.2 mm
- net Net-(J1-Pin_2): track 0.00 -> 19.4 mm
- net Net-(J1-Pin_4): track 0.00 -> 19.3 mm
- net Net-(J8-Pin_8): track 0.00 -> 14.3 mm
- net Net-(J8-Pin_10): track 0.00 -> 8.84 mm
- net Net-(J8-Pin_2): track 0.00 -> 6.61 mm
- net Net-(J8-Pin_6): track 0.00 -> 5.60 mm
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Other:
- board size 65 x 56 mm -> 65 x 23.5 mm
- board text removed: "CAMERA (OPTIONAL)"
- board text removed: "DISPLAY (OPTIONAL)"
- board text removed: "Extend PCB edge 0.5mm if using SMT header"
- board text removed: "PoE"
- board text removed: "RJ45"
- board text removed: "USB"

Commit message: silly
Other:
- board size 65 x 23.5 mm -> 65 x 25.5 mm
- board text added: "EXT1"
- board text added: "GND"
Changed lines of the file:
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@@
 	)
 	(gr_arc
-		(start 165 64)
-		(mid 163.974874 66.474874)
-		(end 161.5 67.5)
+		(start 164.974874 66.025126)
+		(mid 163.957107 68.482233)
+		(end 161.5 69.5)
 		(stroke
 			(width 0.05)
@@
 	)
 	(gr_arc
-		(start 103.5 67.5)
-		(mid 101.025126 66.474874)
-		(end 100 64)
+		(start 103.5 69.5)
+		(mid 101.025126 68.474874)
+		(end 100 66)
 		(stroke
 			(width 0.05)
@@
 	)
 	(gr_line
-		(start 165 64)
+		(start 164.974874 66.025126)
 		(end 165 47)
 		(stroke
@@
 	(gr_line
 		(start 100 53.5)
-		(end 100 64)
+		(end 100 66)
 		(stroke
 			(width 0.1)
@@
 	)
 	(gr_line
-		(start 103.5 67.5)
-		(end 161.5 67.5)
+		(start 103.5 69.5)
+		(end 161.5 69.5)
 		(stroke
 			(width 0.05)
@@
 		(layer "Edge.Cuts")
 	)
+	(gr_text "GND"
+		(at 136 69 0)
+		(layer "F.SilkS")
+		(effects
+			(font
+				(size 0.5 0.5)
+				(thickness 0.1)
+				(bold yes)
+			)
+			(justify left bottom)
+		)
+	)
+	(gr_text "EXT1"
+		(at 111 69 0)
+		(layer "F.SilkS")
+		(effects
+			(font
+				(size 0.5 0.5)
+				(thickness 0.1)
+				(bold yes)
+			)
+			(justify left bottom)
+		)
+	)
 	(segment
